File: cad/Alloy.sch (EAGLE design)
At the start: 71 parts, among them IC1 SPX3819M5_1_2, IC2 MCP73831, IC3 ESP32-S2, IC4 ICE40UP5K, IC5 USBLC6-2SC6, IC6 3.3V, IC7 LY68LXXXX, IC8 AT25SDF041A, Y2 12MZ

Commit message: Added the schematic image
Other:
- note added: "Copyright Alan Wood 2020 @folknology www.mystorm.uk"
Changed lines of the file:
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@@
 <sheet>
 <plain>
+<text x="152.4" y="-81.28" size="2.286" layer="91">Copyright Alan Wood 2020
+@folknology www.mystorm.uk</text>
 </plain>
 <instances>
@@
 </schematic>
 </drawing>
+<compatibility>
+<note version="6.3" minversion="6.2.2" severity="warning">
+Since Version 6.2.2 text objects can contain more than one line,
+which will not be processed correctly with this version.
+</note>
+</compatibility>
 </eagle>
